File: APRSTracker.brd (EAGLE design)
At the start: 100 x 80 mm, 32 parts, among them IC2 TP4056, X1 POWERSUPPLY_DC21MMX

Commit message: brd v1
Parts:
- moved ANT1 72.8 mm to (0.00, 76.2)
- moved SW 71.9 mm to (3.81, 58.4), turned to 180 degrees
- moved X1 70.8 mm to (2.54, 39.4), turned to 90 degrees
- moved ANT 65.0 mm to (0.00, 67.3), turned to 90 degrees
- moved BAT 63.2 mm to (3.81, 50.8), turned to 180 degrees
- moved ICSP 54.0 mm to (81.3, 52.1)
- moved R2 51.1 mm to (58.4, 61.0), turned to 270 degrees
- moved D1 48.3 mm to (55.9, 61.0), turned to 90 degrees
- moved DRA818V 46.6 mm to (26.7, 66.0), turned to 180 degrees
- moved S1 45.7 mm to (52.1, 73.7), turned to 180 degrees
- moved C4 44.0 mm to (13.3, 45.1)
- moved R3 43.3 mm to (50.8, 61.0)
- moved C1 41.6 mm to (58.4, 73.7), turned to 270 degrees
- moved C2 39.5 mm to (55.9, 44.5), turned to 270 degrees
- moved C3 39.5 mm to (55.9, 49.5), turned to 270 degrees
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Connections:
- net GND: now also LED1.K; no longer R4.1
- net LED: now also R4.2; no longer LED1.A
- net N$3: now also LED1.A, R4.1; no longer LED1.K, R4.2
Routing:
- net GND: track 30.5 -> 431.6 mm
- net VCC: track 17.8 -> 392.1 mm
- net V-BAT: track 0.00 -> 367.6 mm
- net CHG: track 0.00 -> 308.9 mm, vias 0 -> 1
- net RF-RX: track 0.00 -> 112.4 mm
- net RF-TX: track 0.00 -> 108.0 mm
- net RESET: track 0.00 -> 76.8 mm
- net VD: track 0.00 -> 73.7 mm, vias 0 -> 1
- net PD2: track 0.00 -> 57.2 mm
- net PD4: track 0.00 -> 52.8 mm
- net N$7: track 0.00 -> 44.4 mm
- net PD3: track 0.00 -> 42.6 mm, vias 0 -> 1
- net N$4: track 0.00 -> 26.7 mm
- net N$1: track 0.00 -> 26.0 mm
- net N$6: track 11.7 -> 33.5 mm
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- added copper zone on layer 16, net GND
Other:
- board size 100 x 80 mm -> 96.2 x 54.6 mm

Commit message: brd update
Routing:
- net GND: track 431.6 -> 152.4 mm
- net CHG: track 308.9 -> 285.1 mm, vias 1 -> 0
- net N$27: track 0.00 -> 7.62 mm
- net N$26: track 0.00 -> 7.62 mm
- net N$24: track 0.00 -> 7.62 mm
- net N$20: track 0.00 -> 7.62 mm
- net N$19: track 0.00 -> 7.62 mm
- net N$15: track 0.00 -> 7.62 mm
- net N$14: track 0.00 -> 7.62 mm
- net N$12: track 0.00 -> 7.62 mm
- net N$25: track 0.00 -> 7.62 mm
- net N$23: track 0.00 -> 7.62 mm
- net N$22: track 0.00 -> 7.62 mm
- net N$21: track 0.00 -> 7.62 mm
- net N$18: track 0.00 -> 7.62 mm
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- added copper zone on layer 1, net GND
Other:
- board size 96.2 x 54.6 mm -> 94.9 x 59.7 mm
- board text added: "+"
- board text added: "APRS Tracker"
- board text added: "Mirzet Brkic | ETF UNSA | 2016."
- board text added: "PB0"
- board text added: "PC1"

Commit message: sch & brd update
Parts:
- removed ICSP: 3x2 M, SmartPrj:2X03
- added ISP: 3x2 M, SmartPrj:2X03
- moved PWR 2.54 mm to (83.8, 74.9)
- turned D1 to 270 degrees
- turned D2 to 90 degrees
- renumbered ANT to SMA
Connections:
- net GND: now also D2.C, ISP.6; no longer D2.A, ICSP.6
- net GPS-RX: no longer D1.C
- net N$2: now also D1.C
- net PB3/MOSI: now also ISP.4; no longer ICSP.4
- net PB4/MISO: now also ISP.1; no longer ICSP.1
- net PB5/SCK: now also ISP.3; no longer ICSP.3
- net RESET: now also ISP.5; no longer ICSP.5
- net VCC: now also ISP.2; no longer ICSP.2
- net VD: now also D2.A; no longer D2.C
Routing:
- net GND: track 152.4 -> 141.6 mm
- net VCC: track 392.6 -> 397.8 mm
- net GPS-RX: track 20.3 -> 15.2 mm
- net RESET: track 76.8 -> 79.3 mm
- net N$2: track 20.3 -> 22.9 mm
- net PB3/MOSI: track 22.9 -> 25.4 mm
- net PB5/SCK: track 31.8 -> 33.0 mm
- net PB4/MISO: track 25.4 -> 26.7 mm
Other:
- board text added: "SMA"
