File: APRSTracker.sch (EAGLE design)
At the start: 26 parts, among them IC1 TP4056

Commit message: sch update
Parts:
- removed PUNJAC: (no value), jumper:JP1E
- added JP1: (no value), jumper:JP1E
- added X1: POWERSUPPLY_DC21MMX, SmartPrj:POWERSUPPLY_DC21MMX
Connections:
- new net N$31: BATERIJA.2, C4.1, IC1.BAT, JP1.1
- net GND: now also X1.1, X1.3; no longer PUNJAC.2
- net N$27: now also X1.2; no longer PUNJAC.1
- net VCC: now also JP1.2; no longer BATERIJA.2, C4.1, IC1.BAT
Other:
- note removed: "mini/micro USB?"
- moved on the sheet: BATERIJA
Changed lines of the file:
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@@
 <class number="0" name="default" width="0" drill="0">
+</class>
+<class number="1" name="power" width="0.6096" drill="0.6096">
+<clearance class="1" value="0.254"/>
 </class>
 <class number="2" name="gnd" width="0.3048" drill="0.5588">
@@
 <part name="C5" library="rcl" deviceset="C-EU" device="050-024X044" value="1u"/>
 <part name="BATERIJA" library="jumper" deviceset="JP1E" device=""/>
-<part name="P+6" library="supply1" deviceset="VCC" device=""/>
 <part name="GND6" library="supply1" deviceset="GND" device=""/>
-<part name="PUNJAC" library="jumper" deviceset="JP1E" device=""/>
 <part name="GND10" library="supply1" deviceset="GND" device=""/>
-<part name="GND11" library="supply1" deviceset="GND" device=""/>
 <part name="GND12" library="supply1" deviceset="GND" device=""/>
-<part name="P+7" library="supply1" deviceset="VCC" device=""/>
 <part name="GND13" library="supply1" deviceset="GND" device=""/>
 <part name="GND14" library="supply1" deviceset="GND" device=""/>
@@
 <part name="ANALOG" library="pinhead" deviceset="PINHD-1X5" device=""/>
 <part name="DIGITAL" library="pinhead" deviceset="PINHD-1X6" device=""/>
+<part name="GND19" library="supply1" deviceset="GND" device=""/>
+<part name="X1" library="SmartPrj" deviceset="POWERSUPPLY_DC21MM" device="X"/>
+<part name="JP1" library="jumper" deviceset="JP1E" device=""/>
+<part name="P+9" library="supply1" deviceset="VCC" device=""/>
 </parts>
 <sheets>
@@
 <text x="60.96" y="99.06" size="1.9304" layer="95">OSCILATOR</text>
 <text x="60.96" y="139.7" size="1.9304" layer="95">RESET</text>
-<text x="226.06" y="96.52" size="1.9304" layer="95">mini/micro USB?</text>
 </plain>
 <instances>
@@
 <instance part="C4" gate="G$1" x="261.62" y="45.72"/>
 <instance part="C5" gate="G$1" x="218.44" y="78.74"/>
-<instance part="BATERIJA" gate="A" x="302.26" y="68.58"/>
-<instance part="P+6" gate="VCC" x="304.8" y="58.42" rot="R180"/>
+<instance part="BATERIJA" gate="A" x="302.26" y="73.66"/>
 <instance part="GND6" gate="1" x="302.26" y="58.42"/>
-<instance part="PUNJAC" gate="A" x="226.06" y="86.36"/>
 <instance part="GND10" gate="1" x="215.9" y="45.72"/>
-<instance part="GND11" gate="1" x="228.6" y="78.74"/>
 <instance part="GND12" gate="1" x="228.6" y="58.42" rot="R270"/>
-<instance part="P+7" gate="VCC" x="271.78" y="50.8" rot="R270"/>
 <instance part="GND13" gate="1" x="261.62" y="35.56"/>
 <instance part="GND14" gate="1" x="218.44" y="68.58"/>
@@
 <instance part="ANALOG" gate="A" x="147.32" y="96.52"/>
 <instance part="DIGITAL" gate="A" x="147.32" y="76.2"/>
+<instance part="GND19" gate="1" x="256.54" y="101.6"/>
+<instance part="X1" gate="G$1" x="261.62" y="124.46" smashed="yes">
+<attribute name="NAME" x="251.46" y="132.08" size="1.27" layer="94"/>
+<attribute name="VALUE" x="251.46" y="129.54" size="1.27" layer="94"/>
+</instance>
+<instance part="JP1" gate="A" x="314.96" y="73.66"/>
+<instance part="P+9" gate="VCC" x="317.5" y="33.02" rot="R180"/>
 </instances>
 <busses>
@@
 <pinref part="BATERIJA" gate="A" pin="1"/>
 <pinref part="GND6" gate="1" pin="GND"/>
-<wire x1="302.26" y1="60.96" x2="302.26" y2="66.04" width="0.1524" layer="91"/>
+<wire x1="302.26" y1="60.96" x2="302.26" y2="71.12" width="0.1524" layer="91"/>
 </segment>
 <segment>
@@
 <pinref part="GND14" gate="1" pin="GND"/>
 <wire x1="218.44" y1="71.12" x2="218.44" y2="73.66" width="0.1524" layer="91"/>
-</segment>
-<segment>
-<pinref part="PUNJAC" gate="A" pin="2"/>
-<pinref part="GND11" gate="1" pin="GND"/>
-<wire x1="228.6" y1="81.28" x2="228.6" y2="83.82" width="0.1524" layer="91"/>
 </segment>
 <segment>
@@
 <pinref part="GND8" gate="1" pin="GND"/>
 <wire x1="187.96" y1="40.64" x2="187.96" y2="45.72" width="0.1524" layer="91"/>
+</segment>
+<segment>
+<wire x1="256.54" y1="114.3" x2="256.54" y2="109.22" width="0.1524" layer="91"/>
+<wire x1="256.54" y1="109.22" x2="256.54" y2="104.14" width="0.1524" layer="91"/>
+<wire x1="256.54" y1="109.22" x2="276.86" y2="109.22" width="0.1524" layer="91"/>
+<wire x1="276.86" y1="109.22" x2="276.86" y2="124.46" width="0.1524" layer="91"/>
+<wire x1="256.54" y1="106.68" x2="256.54" y2="109.22" width="0.1524" layer="91"/>
+<junction x="256.54" y="109.22"/>
+<pinref part="X1" gate="G$1" pin="1"/>
+<pinref part="GND19" gate="1" pin="GND"/>
+<pinref part="X1" gate="G$1" pin="3"/>
 </segment>
 </net>
@@
 <net name="VCC" class="0">
 <segment>
-<pinref part="BATERIJA" gate="A" pin="2"/>
-<pinref part="P+6" gate="VCC" pin="VCC"/>
-<wire x1="304.8" y1="60.96" x2="304.8" y2="66.04" width="0.1524" layer="91"/>
-</segment>
-<segment>
-<pinref part="IC1" gate="G$1" pin="BAT"/>
-<pinref part="C4" gate="G$1" pin="1"/>
-<wire x1="261.62" y1="55.88" x2="261.62" y2="50.8" width="0.1524" layer="91"/>
-<pinref part="P+7" gate="VCC" pin="VCC"/>
-<wire x1="261.62" y1="50.8" x2="261.62" y2="48.26" width="0.1524" layer="91"/>
-<wire x1="269.24" y1="50.8" x2="261.62" y2="50.8" width="0.1524" layer="91"/>
-</segment>
-<segment>
 <pinref part="R1" gate="G$1" pin="2"/>
 <wire x1="81.28" y1="139.7" x2="81.28" y2="132.08" width="0.1524" layer="91"/>
@@
 <wire x1="187.96" y1="78.74" x2="187.96" y2="73.66" width="0.1524" layer="91"/>
 </segment>
+<segment>
+<pinref part="JP1" gate="A" pin="2"/>
+<pinref part="P+9" gate="VCC" pin="VCC"/>
+<wire x1="317.5" y1="35.56" x2="317.5" y2="71.12" width="0.1524" layer="91"/>
+</segment>
 </net>
 <net name="N$18" class="0">
@@
 <wire x1="233.68" y1="55.88" x2="226.06" y2="55.88" width="0.1524" layer="91"/>
 <wire x1="226.06" y1="55.88" x2="226.06" y2="71.12" width="0.1524" layer="91"/>
-<pinref part="PUNJAC" gate="A" pin="1"/>
 <wire x1="226.06" y1="71.12" x2="226.06" y2="81.28" width="0.1524" layer="91"/>
 <pinref part="IC1" gate="G$1" pin="CE"/>
-<wire x1="226.06" y1="81.28" x2="226.06" y2="83.82" width="0.1524" layer="91"/>
 <wire x1="261.62" y1="63.5" x2="261.62" y2="71.12" width="0.1524" layer="91"/>
 <wire x1="261.62" y1="71.12" x2="226.06" y2="71.12" width="0.1524" layer="91"/>
@@
 <pinref part="C5" gate="G$1" pin="1"/>
 <wire x1="218.44" y1="81.28" x2="226.06" y2="81.28" width="0.1524" layer="91"/>
+<pinref part="X1" gate="G$1" pin="2"/>
+<wire x1="266.7" y1="114.3" x2="226.06" y2="114.3" width="0.1524" layer="91"/>
+<wire x1="226.06" y1="114.3" x2="226.06" y2="81.28" width="0.1524" layer="91"/>
 </segment>
 </net>
@@
 </segment>
 </net>
+<net name="N$31" class="0">
+<segment>
+<pinref part="IC1" gate="G$1" pin="BAT"/>
+<pinref part="C4" gate="G$1" pin="1"/>
+<wire x1="261.62" y1="55.88" x2="261.62" y2="50.8" width="0.1524" layer="91"/>
+<wire x1="261.62" y1="50.8" x2="261.62" y2="48.26" width="0.1524" layer="91"/>
+<pinref part="BATERIJA" gate="A" pin="2"/>
+<wire x1="304.8" y1="71.12" x2="304.8" y2="66.04" width="0.1524" layer="91"/>
+<wire x1="304.8" y1="66.04" x2="309.88" y2="66.04" width="0.1524" layer="91"/>
+<pinref part="JP1" gate="A" pin="1"/>
+<wire x1="309.88" y1="66.04" x2="314.96" y2="66.04" width="0.1524" layer="91"/>
+<wire x1="314.96" y1="66.04" x2="314.96" y2="71.12" width="0.1524" layer="91"/>
+<wire x1="261.62" y1="50.8" x2="309.88" y2="50.8" width="0.1524" layer="91"/>
+<wire x1="309.88" y1="50.8" x2="309.88" y2="66.04" width="0.1524" layer="91"/>
+</segment>
+</net>

Commit message: shema v2
Parts:
- removed ANALOG: (no value), pinhead:PINHD-1X5
- removed BATERIJA, JP1: (no value), jumper:JP1E
- removed C6: 100n, rcl:C-EU050-024X044
- removed DIGITAL: (no value), pinhead:PINHD-1X6
- removed IC1: TP4056, TP4056:TP4056
- removed LED5, LED6: (no value), led:LED3MM
- removed R10: 2k2, rcl:R-EU_0207/10
- added ANT: SMA_EDGE, SparkFun:SMA_EDGE
- added BAT, SW: (no value), jumper:JP1E
- added D2: 1N4004, diode1:1N4004
- added IC2: TP4056, TP4056:TP4056
- added LED1, LED2, LED3: (no value), led:LED3MM
- added PORTB: (no value), pinhead:PINHD-1X6
- added PORTC: (no value), pinhead:PINHD-1X5
- added PWR: (no value), pinhead:PINHD-2X3
- added R5, R6: 1k, rcl:R-EU_0207/10
- added R7: 2k2, rcl:R-EU_0207/10
- D1: value 1N4004 -> (none); device diode:1N4004 -> diode:ZENER-DIODEDO35Z10
- R2: value 10k -> (none)
- R3: value 1k -> 10k
- R4: value 1k -> 330
Connections:
- net N$4 renamed RESET
- removed net N$10: ANT1.1, DRA818V.ANT
- removed net N$11: DRA818V.TXD, MCU.(OC1)PB1
- removed net N$12: DRA818V.RXD, MCU.(ICP)PB0
- removed net N$13: ANALOG.1, MCU.(ADC5)PC5
- removed net N$14: D1.C, MCU.(ADC0)PC0), R2.1
- removed net N$15: ANALOG.2, MCU.(ADC4)PC4
- removed net N$16: ANALOG.3, MCU.(ADC3)PC3
- removed net N$17: ANALOG.4, MCU.(ADC2)PC2
- removed net N$18: IC1.CHRG, R4.1
- removed net N$19: ANALOG.5, MCU.(ADC1)PC1
- removed net N$20: DIGITAL.1, MCU.(AIN1)PD7
- removed net N$21: DIGITAL.2, MCU.(AIN0)PD6
- removed net N$22: DIGITAL.3, MCU.(T1)PD5
- removed net N$23: IC1.STDBY, R3.2
- removed net N$24: LED5.C, R4.2
- removed net N$25: LED6.C, R3.1
- removed net N$26: IC1.PROG, R10.2
- removed net N$27: C5.1, IC1.CE, IC1.VCC, LED5.A, LED6.A, X1.2
- removed net N$28: DIGITAL.4, MCU.(T0)PD4
- removed net N$29: DIGITAL.5, MCU.(INT1)PD3
- removed net N$30: DIGITAL.6, MCU.(INT0)PD2
- removed net N$31: BATERIJA.2, C4.1, IC1.BAT, JP1.1
- removed net N$8: GPS.3, MCU.(RXD)PD0
- removed net N$9: DRA818V.MIC, MCU.(SS)PB2
- new net CHG: C5.1, IC2.CE, IC2.VCC, LED2.A, LED3.A, X1.2
- new net GPS-RX: D1.C, MCU.(TXD)PD1, R2.2
- new net GPS-TX: GPS.2, MCU.(RXD)PD0
- new net LED: LED1.A, MCU.(AIN1)PD7
- new net LED1: IC2.CHRG, R5.1
- new net LED2: IC2.STDBY, R6.1
- new net N$4: LED2.C, R5.2
- new net PB0: MCU.(ICP)PB0, PORTB.1
- new net PB1: MCU.(OC1)PB1, PORTB.2
- new net PB2: MCU.(SS)PB2, PORTB.3
- new net PB3/MOSI: ICSP.4, MCU.(MOSI)PB3, PORTB.4
- new net PB4/MISO: ICSP.1, MCU.(MISO)PB4, PORTB.5
- new net PB5/SCK: ICSP.3, MCU.(SCK)PB5, PORTB.6
- new net PC1: MCU.(ADC1)PC1, PORTC.1
- new net PC2: MCU.(ADC2)PC2, PORTC.2
- new net PC3: MCU.(ADC3)PC3, PORTC.3
- new net PC4: MCU.(ADC4)PC4, PORTC.4
- new net PC5: MCU.(ADC5)PC5, PORTC.5
- new net PD2: DRA818V.PD, MCU.(INT0)PD2
- new net PD3: DRA818V.MIC, MCU.(INT1)PD3
- new net PD4: DRA818V.PTT, MCU.(T0)PD4
- new net PROG: IC2.PROG, R7.1
- new net RF-RX: DRA818V.RXD, MCU.(AIN0)PD6
- new net RF-TX: DRA818V.TXD, MCU.(T1)PD5
- new net V-BAT: BAT.1, C4.1, IC2.BAT, SW.2
- new net VD: D2.C, MCU.(ADC0)PC0), R3.1
- net GND: now also ANT.GND@0, ANT.GND@1, ANT.GND@2, ANT.GND@3, BAT.2, D1.A, D2.A, GPS.1, IC2.GND, IC2.TEMP, PWR.1, PWR.3, PWR.5, R4.1, R7.2; no longer BATERIJA.1, C6.1, GPS.4, IC1.GND, IC1.TEMP, R10.1, R2.2
- net N$1: now also ANT.SIGNAL, ANT1.1, DRA818V.ANT; no longer ICSP.4, MCU.(MOSI)PB3
- net N$2: now also GPS.3, R2.1; no longer DRA818V.PD, ICSP.1, MCU.(MISO)PB4
- net N$3: now also LED1.C, R4.2; no longer DRA818V.PTT, ICSP.3, MCU.(SCK)PB5
- net N$7: now also LED3.C, R6.2; no longer GPS.2, MCU.(TXD)PD1
- net VCC: now also GPS.4, PWR.2, PWR.4, PWR.6, R3.2, SW.1; no longer C6.2, D1.A, GPS.1, JP1.2
Other:
- note added: "GPIO"
- note added: "GPS"
- note added: "ICSP"
- note added: "MICROCONTROLLER"
- note added: "POWER"
- note added: "RF"
- note added: "V-BAT"
- note removed: "OSCILATOR"
- note removed: "RESET"
- moved on the sheet: ANT1, C1, C2, C3, C4, C5, DRA818V, GPS, ICSP, MCU, Q1, R1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

Commit message: brd v1
Connections:
- net GND: now also LED1.C; no longer R4.1
- net LED: now also R4.2; no longer LED1.A
- net N$3: now also LED1.A, R4.1; no longer LED1.C, R4.2
Other:
- moved on the sheet: C5, LED1, R4
Changed lines of the file:
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@@
 <part name="GND13" library="supply1" deviceset="GND" device=""/>
 <part name="GND15" library="supply1" deviceset="GND" device=""/>
-<part name="GND17" library="supply1" deviceset="GND" device=""/>
 <part name="GND18" library="supply1" deviceset="GND" device=""/>
 <part name="R6" library="rcl" deviceset="R-EU_" device="0207/10" value="1k"/>
@@
 <part name="GND20" library="supply1" deviceset="GND" device=""/>
 <part name="P+8" library="supply1" deviceset="VCC" device=""/>
+<part name="GND17" library="supply1" deviceset="GND" device=""/>
 </parts>
 <sheets>
@@
 <instance part="R2" gate="G$1" x="50.8" y="167.64"/>
 <instance part="D1" gate="G$1" x="58.42" y="162.56" rot="R90"/>
-<instance part="GND11" gate="1" x="58.42" y="157.48"/>
+<instance part="GND11" gate="1" x="58.42" y="154.94"/>
 <instance part="R3" gate="G$1" x="167.64" y="66.04" rot="R90"/>
 <instance part="D2" gate="1" x="167.64" y="50.8" smashed="yes" rot="R90">
@@
 <instance part="R5" gate="G$1" x="106.68" y="137.16"/>
 <instance part="R7" gate="G$1" x="109.22" y="121.92"/>
-<instance part="C5" gate="G$1" x="154.94" y="170.18"/>
+<instance part="C5" gate="G$1" x="154.94" y="172.72"/>
 <instance part="BAT" gate="A" x="124.46" y="190.5" smashed="yes">
 <attribute name="NAME" x="127.762" y="195.58" size="1.778" layer="95" rot="R180"/>
@@
 <attribute name="VALUE" x="106.68" y="149.86" size="1.778" layer="96"/>
 </instance>
-<instance part="GND17" gate="1" x="154.94" y="162.56"/>
 <instance part="GND18" gate="1" x="111.76" y="154.94" smashed="yes" rot="R270">
 <attribute name="VALUE" x="106.68" y="154.94" size="1.778" layer="96"/>
@@
 <instance part="FRAME1" gate="G$1" x="0" y="2.54"/>
 <instance part="PORTB" gate="A" x="157.48" y="231.14"/>
-<instance part="LED1" gate="G$1" x="142.24" y="66.04"/>
-<instance part="R4" gate="G$1" x="142.24" y="50.8" rot="R90"/>
+<instance part="LED1" gate="G$1" x="142.24" y="53.34"/>
+<instance part="R4" gate="G$1" x="142.24" y="66.04" rot="R90"/>
 <instance part="GND19" gate="1" x="142.24" y="38.1" smashed="yes">
 <attribute name="VALUE" x="142.24" y="35.56" size="1.778" layer="96"/>
@@
 <instance part="GND20" gate="1" x="142.24" y="127" rot="R270"/>
 <instance part="P+8" gate="VCC" x="170.18" y="132.08" rot="R270"/>
+<instance part="GND17" gate="1" x="154.94" y="162.56"/>
 </instances>
 <busses>
@@
 <pinref part="D1" gate="G$1" pin="A"/>
 <pinref part="GND11" gate="1" pin="GND"/>
+<wire x1="58.42" y1="157.48" x2="58.42" y2="160.02" width="0.1524" layer="91"/>
 </segment>
 <segment>
@@
 </segment>
 <segment>
-<pinref part="C5" gate="G$1" pin="2"/>
-<pinref part="GND17" gate="1" pin="GND"/>
-</segment>
-<segment>
 <pinref part="IC2" gate="G$1" pin="TEMP"/>
 <pinref part="GND18" gate="1" pin="GND"/>
@@
 <pinref part="GND16" gate="1" pin="GND"/>
 <wire x1="124.46" y1="165.1" x2="124.46" y2="167.64" width="0.1524" layer="91"/>
-</segment>
-<segment>
-<pinref part="R4" gate="G$1" pin="1"/>
-<pinref part="GND19" gate="1" pin="GND"/>
-<wire x1="142.24" y1="45.72" x2="142.24" y2="40.64" width="0.1524" layer="91"/>
 </segment>
 <segment>
@@
 <pinref part="PWR" gate="A" pin="5"/>
 <wire x1="152.4" y1="127" x2="147.32" y2="127" width="0.1524" layer="91"/>
+</segment>
+<segment>
+<pinref part="C5" gate="G$1" pin="2"/>
+<pinref part="GND17" gate="1" pin="GND"/>
+<wire x1="154.94" y1="165.1" x2="154.94" y2="167.64" width="0.1524" layer="91"/>
+</segment>
+<segment>
+<pinref part="GND19" gate="1" pin="GND"/>
+<pinref part="LED1" gate="G$1" pin="C"/>
+<wire x1="142.24" y1="48.26" x2="142.24" y2="40.64" width="0.1524" layer="91"/>
 </segment>
 </net>
@@
 <segment>
 <pinref part="X1" gate="G$1" pin="2"/>
-<wire x1="154.94" y1="177.8" x2="154.94" y2="172.72" width="0.1524" layer="91"/>
+<wire x1="154.94" y1="177.8" x2="154.94" y2="175.26" width="0.1524" layer="91"/>
 <label x="157.48" y="175.26" size="1.778" layer="95" rot="R90"/>
 <pinref part="C5" gate="G$1" pin="1"/>
@@
 </segment>
 <segment>
-<pinref part="LED1" gate="G$1" pin="A"/>
-<wire x1="142.24" y1="68.58" x2="142.24" y2="76.2" width="0.1524" layer="91"/>
+<pinref part="R4" gate="G$1" pin="2"/>
+<wire x1="142.24" y1="71.12" x2="142.24" y2="76.2" width="0.1524" layer="91"/>
 <label x="142.24" y="73.66" size="1.778" layer="95" rot="R90"/>
 </segment>
@@
 <net name="N$3" class="0">
 <segment>
-<pinref part="LED1" gate="G$1" pin="C"/>
-<pinref part="R4" gate="G$1" pin="2"/>
-<wire x1="142.24" y1="60.96" x2="142.24" y2="55.88" width="0.1524" layer="91"/>
-</segment>
-</net>
+<pinref part="LED1" gate="G$1" pin="A"/>
+<pinref part="R4" gate="G$1" pin="1"/>
+<wire x1="142.24" y1="55.88" x2="142.24" y2="60.96" width="0.1524" layer="91"/>
+</segment>
+</net>

Commit message: power
Other:
- note added: "SMA"
Changed lines of the file:
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@@
 <?xml version="1.0" encoding="utf-8"?>
 <!DOCTYPE eagle SYSTEM "eagle.dtd">
-<eagle version="7.5.0">
+<eagle version="7.6.0">
 <drawing>
 <settings>
@@
 <text x="35.56" y="88.9" size="5.08" layer="95">MICROCONTROLLER</text>
 <wire x1="119.38" y1="106.68" x2="119.38" y2="2.54" width="0.1524" layer="95" style="longdash"/>
+<text x="73.66" y="223.52" size="1.778" layer="95" rot="R90">SMA</text>
 </plain>
 <instances>

Commit message: sch & brd update
Parts:
- renumbered ANT to SMA, ICSP to ISP
Connections:
- net GND: now also D2.C; no longer D2.A
- net GPS-RX: no longer D1.C
- net N$2: now also D1.C
- net VD: now also D2.A; no longer D2.C
Other:
- note added: "GY-NEO6MV2"
- note added: "ISP"
- note added: "Mirzet Brkic, ETF UNSA 2016.g."
- note removed: "ICSP"
- moved on the sheet: ANT1, D1, D2, R2
